File: pcb/half-swept.kicad_sch (KiCad schematic)
At the start: 60 parts, among them J1 AudioJack4dpb, J2 AudioJack4dpb, SW1 SW_Push, SW10 SW_Push, SW11 SW_Push, SW12 SW_Push, SW14 SW_Push, SW15 SW_Push, SW16 SW_Push, SW17 SW_Push, SW18 SW_Push, SW2 SW_Push, SW20 SW_Push, SW21 SW_Push, SW3 SW_Push, SW4 SW_Push, SW5 SW_Push, SW6 SW_Push, SW8 SW_Push, SW9 SW_Push, U2 Elite-C

Commit message: converted to choc reversible hotswap
Parts:
- SW1, SW10, SW11, SW12, SW14, SW15, SW16, SW17, SW18, SW2, SW20, SW21, SW3, SW4, SW5, SW6, SW8, SW9: footprint Keebio-Parts:Kailh-PG1350-1u-reversible -> keyswitches:Kailh_socket_PG1350_reversible
